File: UGVboard.brd (EAGLE design)
At the start: 101.3 x 53.3 mm, 44 parts, among them IC1 NE555D, IC2 NE555D, U1 L3G4200D

Commit message: Updates to Board for v1.2
Parts:
- renumbered U1 to GYROSCOPE
Connections:
- net N$1 renamed D52
- net N$10 renamed SCL1
- net N$11 renamed D2
- net N$12 renamed D3
- net N$13 renamed D27
- net N$14 renamed D29
- net N$2 renamed D44
- net N$3 renamed D51
- net N$30 renamed D30
- net N$31 renamed D25
- net N$32 renamed D28
- net N$39 renamed RST
- net N$4 renamed D26
- net N$43 renamed A2
- net N$44 renamed A3
- net N$45 renamed A4
- net N$46 renamed A5
- net N$5 renamed D53
- net N$6 renamed SCK
- net N$7 renamed SDA1
- net N$8 renamed SS1
- net N$9 renamed D83
- removed net VSS: SDCARD.6, SDCARD.MT1, SDCARD.MT2
- new net VDD: SDCARD.4
- net 3.3V: now also GYROSCOPE.4, GYROSCOPE.5; no longer SDCARD.4
- net GND: now also SDCARD.6, SDCARD.MT1, SDCARD.MT2
Routing:
- net VSS: track 31.2 -> 0.00 mm, vias 2 -> 0
- net GND: track 27.6 -> 20.5 mm, vias 19 -> 18
- net 3.3V: track 187.7 -> 192.8 mm
- net D3: track 10.2 -> 10.9 mm
