File: UGVboard.sch (EAGLE design)
At the start: 42 parts, among them IC1 NE555D, IC2 NE555D, U1 L3G4200D

Commit message: Updates to Board for v1.2
Parts:
- removed U1: L3G4200D, SparkFun:L3G4200D
- added GYROSCOPE: L3G4200D, SparkFun:L3G4200D
Connections:
- net N$1 renamed D52
- net N$10 renamed SCL1
- net N$11 renamed D2
- net N$12 renamed D3
- net N$13 renamed D27
- net N$14 renamed D29
- net N$2 renamed D44
- net N$3 renamed D51
- net N$30 renamed D30
- net N$31 renamed D25
- net N$32 renamed D28
- net N$39 renamed RST
- net N$4 renamed D26
- net N$43 renamed A2
- net N$44 renamed A3
- net N$45 renamed A4
- net N$46 renamed A5
- net N$5 renamed D53
- net N$6 renamed SCK
- net N$7 renamed SDA1
- net N$8 renamed SS1
- net N$9 renamed D83
- removed net VSS: SDCARD.GND, SDCARD.GND1, SDCARD.VSS
- new net VDD: SDCARD.VDD
- net 3.3V: now also GYROSCOPE.CS, GYROSCOPE.RSVDV@0, GYROSCOPE.SDO, GYROSCOPE.VDD, GYROSCOPE.VDDIO; no longer SDCARD.VDD, U1.RSVDV@0, U1.VDD, U1.VDDIO
- net GND: now also GYROSCOPE.GND, GYROSCOPE.RSDVG@3, GYROSCOPE.RSVDG@0, GYROSCOPE.RSVDG@1, GYROSCOPE.RSVDG@2, GYROSCOPE.RSVDG@4, SDCARD.GND, SDCARD.GND1, SDCARD.VSS; no longer U1.GND, U1.RSDVG@3, U1.RSVDG@0, U1.RSVDG@1, U1.RSVDG@2, U1.RSVDG@4
- net PLL: now also GYROSCOPE.PLL; no longer U1.PLL
- net SCL: now also GYROSCOPE.SCL; no longer U1.SCL
- net SDA: now also GYROSCOPE.SDA/SDI; no longer U1.SDA/SDI
Other:
- note removed: "1.2"
- moved on the sheet: C1, C2, C3, C4, C5, D1, EN1, EN2, GPS, IC1, IC2, JP1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
